File: canon+GH4.kicad_pcb (KiCad board)
At the start: 2 copper layers, 28.5 x 35.5 mm, 16 parts, among them Q1 2SC1815, Q2 2SC1815, Q3 2SC1815

Commit message: updates
Parts:
- TP5: value F -> S
- TP6: value S -> F
- TP7: value F2 -> S2
- moved TP2 11.1 mm to (117.5, 92.5)
- moved R5 9.48 mm to (127.0, 85.7), turned to -90 degrees
- moved R4 9.43 mm to (129.5, 85.7), turned to -90 degrees
- moved TP3 8.49 mm to (112.5, 92.5)
- moved R6 7.84 mm to (122.5, 91.6), turned to 90 degrees
- moved R3 6.02 mm to (127.5, 71.5), turned to -130 degrees
- moved TP4 5.00 mm to (112.5, 68.0)
- moved R1 3.91 mm to (122.5, 71.5), turned to -130 degrees
- moved TP1 3.35 mm to (108.0, 92.5)
- moved R2 2.88 mm to (117.5, 71.5), turned to -150 degrees
- moved TP6 2.50 mm to (117.5, 68.0)
- moved TP5 1.50 mm to (122.5, 68.0)
- moved TP7 0.50 mm to (127.5, 68.0)
- moved Q2 0.40 mm to (109.9, 81.0)
Connections:
- net /Signal_focus renamed /Focus_Input
- net /Signal_shutter renamed /Shutter_Input
- net Net-(Q2-C) renamed /Focus_Output
- net Net-(R6-Pad1) renamed /Focus_Input_GH4
- Q1 pad 1: /Ground -> GND
- Q1 pad 2: Net-(Q1-C) -> /Shutter_Output
- Q2 pad 1: /Ground -> GND
- Q3 pad 2: Net-(Q1-C) -> /Shutter_Output
- R4 pad 1: /Ground -> Net-(Q3-E)
- R4 pad 2: Net-(Q3-E) -> GND
- R5 pad 1: Net-(R4-Pad1) -> Net-(Q3-E)
- R5 pad 2: Net-(Q3-E) -> Net-(R5-Pad2)
- R6 pad 1: Net-(Q1-C) -> Net-(R5-Pad2)
- R6 pad 2: Net-(R4-Pad1) -> /Shutter_Output
- TP1 pad 1: /Ground -> GND
- TP2 pad 1: Net-(Q1-C) -> /Shutter_Output
- TP4 pad 1: /Ground -> GND
Routing:
- net Net-(Q1-C): track 33.0 -> 0.00 mm
- net /Shutter_Output: track 0.00 -> 27.9 mm
- net Net-(Q3-E): track 16.9 -> 7.19 mm
- net Net-(R4-Pad1): track 9.40 -> 0.00 mm
- net /Focus_Output: track 6.80 -> 13.1 mm
- net /Focus_Input_GH4: track 9.50 -> 3.50 mm
- net Net-(R5-Pad2): track 0.00 -> 5.20 mm
- net /Shutter_Input: track 6.91 -> 3.50 mm
- net Net-(Q3-B): track 9.13 -> 7.50 mm
- net Net-(Q2-B): track 9.52 -> 8.44 mm
- net Net-(Q1-B): track 7.36 -> 6.39 mm
- added copper zone on F.Cu, net GND
- removed copper zone on F.Cu, net /Ground
Other:
- board size 28.5 x 35.5 mm -> 27 x 31 mm

Commit message: a
Parts:
- moved R6 29.8 mm to (101.0, 70.9)
- moved Q2 29.8 mm to (88.4, 60.3)
- moved Q1 29.8 mm to (95.5, 60.3)
- moved Q3 29.8 mm to (108.0, 60.3)
- moved R1 29.8 mm to (101.0, 50.8)
- moved R2 29.8 mm to (96.0, 50.8), turned to -130 degrees
- moved R3 29.8 mm to (106.0, 50.8)
- moved R4 29.8 mm to (108.0, 65.0)
- moved R5 29.8 mm to (105.5, 65.0)
- moved TP1 29.8 mm to (86.5, 71.8)
- moved TP2 29.8 mm to (96.0, 71.8)
- moved TP3 29.8 mm to (91.0, 71.8)
- moved TP4 29.8 mm to (91.0, 47.3)
- moved TP5 29.8 mm to (101.0, 47.3)
- moved TP6 29.8 mm to (96.0, 47.3)
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Other:
- board text added: "${TITLE} ${COMMENT1} (${REVISION})"

Commit message: update
Parts:
- moved Q3 5.73 mm to (102.3, 60.3)
- moved R6 2.24 mm to (102.5, 72.6)
- moved R4 0.50 mm to (108.5, 65.0)
Routing:
- net Net-(Q3-B): track 7.50 -> 4.23 mm
- net Net-(Q3-E): track 7.19 -> 9.93 mm
- net Net-(R5-Pad2): track 5.20 -> 2.54 mm
- net /Shutter_Output: track 27.9 -> 26.7 mm
- net Net-(Q1-B): track 6.39 -> 5.44 mm
Other:
- board text removed: "${TITLE} ${COMMENT1} (${REVISION})"

Commit message: e
Parts:
- removed TP7: S2, TestPoint:TestPoint_THTPad_2.0x2.0mm_Drill1.0mm
- added SW1: SW_DIP_x02, Button_Switch_THT:SW_DIP_SPSTx02_Slide_9.78x7.26mm_W7.62mm_P2.54mm, F.Cu at (97.0, 68.9)
- moved TP1 10.2 mm to (86.5, 82.0)
- moved TP2 10.2 mm to (96.0, 82.0)
- moved TP3 10.2 mm to (91.0, 82.0)
Connections:
- Q1 pad 2: /Shutter_Output -> Net-(Q1-C)
- Q3 pad 2: /Shutter_Output -> Net-(Q3-C)
- R3 pad 1: /Focus_Input_GH4 -> /Shutter_Input
- R6 pad 2: /Shutter_Output -> Net-(Q3-C)
- TP2 pad 1: /Shutter_Output -> Net-(SW1-Pad3)
Routing:
- net /Shutter_Output: track 26.7 -> 0.00 mm
- net Net-(Q3-C): track 0.00 -> 13.2 mm
- net Net-(SW1-Pad3): track 0.00 -> 10.6 mm
- net /Focus_Output: track 13.1 -> 23.3 mm
- net Net-(Q1-C): track 0.00 -> 8.67 mm
- net /Shutter_Input: track 3.50 -> 8.50 mm
- net /Focus_Input_GH4: track 3.50 -> 0.00 mm
Other:
- board size 27 x 31 mm -> 27 x 41.7 mm
