File: canon+GH4.kicad_sch (KiCad schematic)
At the start: 16 parts, among them Q1 2SC1815, Q2 2SC1815, Q3 2SC1815

Commit message: updates
Parts:
- R4, R5, R6: symbol Device:R -> Device:R_US
- TP5: value F -> S
- TP6: value S -> F
- TP7: value F2 -> S2
Connections:
- net Focus_Input_GH4: now reaches R3.1, TP7.1
- net Focus_Output: now reaches Q2.2 (C), TP3.1
- net Shutter_Output: now reaches Q1.2 (C), Q3.2 (C), TP2.1
- net Shutter_Output: now also R6.2; no longer R6.1
- net at R5.1: now also Q3.1 (E), R4.1; no longer R6.2
- net Ground renamed GND
- net GND: now also R4.2; no longer R4.1
- net Signal_focus renamed Focus_Input
- net Signal_shutter renamed Shutter_Input
- new net: R5.2, R6.1
Other:
- moved on the sheet: Q1, Q2, Q3, R1, R2, R3, TP1, TP2, TP3, TP4, TP5, TP6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

Commit message: update
Connections:
- net Focus_Input_GH4 renamed Shutter_Input_GH4
Changed lines of the file:
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@@
 		)
 	)
-	(label "Focus_Input_GH4"
+	(label "Shutter_Input_GH4"
 		(at 132.08 40.64 0)
 		(fields_autoplaced yes)

Commit message: e
Parts:
- removed TP7: S2, TestPoint:TestPoint_THTPad_2.0x2.0mm_Drill1.0mm, symbol Connector:TestPoint
- added SW1: SW_DIP_x02, Button_Switch_THT:SW_DIP_SPSTx02_Slide_9.78x7.26mm_W7.62mm_P2.54mm, symbol Switch:SW_DIP_x02
Connections:
- net Shutter_Input_GH4 is gone; now on net Shutter_Input: R3.1
- net Shutter_Output: no longer Q1.2 (C), Q3.2 (C), R6.2, TP2.1
- new net: Q3.2 (C), R6.2, SW1.1
- new net: Q1.2 (C), SW1.2
- new net: SW1.3, SW1.4, TP2.1
Other:
- moved on the sheet: R5, R6
Changed lines of the file:
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@@
 	(paper "A5")
 	(junction
-		(at 80.01 67.31)
+		(at 128.27 62.23)
 		(diameter 0)
 		(color 0 0 0 0)
 	)
 	(junction
-		(at 57.15 67.31)
+		(at 128.27 40.64)
 		(diameter 0)
 		(color 0 0 0 0)
@@
 	)
 	(junction
+		(at 58.42 64.77)
+		(diameter 0)
+		(color 0 0 0 0)
+	)
+	(junction
+		(at 43.18 67.31)
+		(diameter 0)
+		(color 0 0 0 0)
+	)
+	(junction
 		(at 154.94 22.86)
 		(diameter 0)
@@
 	(wire
 		(pts
-			(xy 57.15 46.99) (xy 57.15 53.34)
-		)
-		(stroke
-			(width 0)
-			(type default)
-		)
-	)
-	(wire
-		(pts
-			(xy 156.21 40.64) (xy 97.79 40.64)
+			(xy 62.23 45.72) (xy 62.23 52.07)
 		)
 		(stroke
@@
 	(wire
 		(pts
-			(xy 35.56 67.31) (xy 57.15 67.31)
+			(xy 128.27 62.23) (xy 157.48 62.23)
 		)
 		(stroke
@@
 	(wire
 		(pts
-			(xy 80.01 45.72) (xy 80.01 67.31)
-		)
-		(stroke
-			(width 0)
-			(type default)
-		)
-	)
-	(wire
-		(pts
 			(xy 110.49 87.63) (xy 115.57 87.63)
 		)
@@
 	(wire
 		(pts
+			(xy 128.27 40.64) (xy 156.21 40.64)
+		)
+		(stroke
+			(width 0)
+			(type default)
+		)
+	)
+	(wire
+		(pts
 			(xy 123.19 87.63) (xy 157.48 87.63)
 		)
@@
 	(wire
 		(pts
+			(xy 58.42 67.31) (xy 104.14 67.31)
+		)
+		(stroke
+			(width 0)
+			(type default)
+		)
+	)
+	(wire
+		(pts
 			(xy 88.9 25.4) (xy 92.71 25.4)
 		)
@@
 	(wire
 		(pts
-			(xy 123.19 62.23) (xy 157.48 62.23)
+			(xy 123.19 62.23) (xy 128.27 62.23)
+		)
+		(stroke
+			(width 0)
+			(type default)
+		)
+	)
+	(wire
+		(pts
+			(xy 43.18 64.77) (xy 43.18 67.31)
 		)
 		(stroke
@@
 	(wire
 		(pts
-			(xy 57.15 60.96) (xy 57.15 67.31)
-		)
-		(stroke
-			(width 0)
-			(type default)
-		)
-	)
-	(wire
-		(pts
-			(xy 80.01 67.31) (xy 104.14 67.31)
-		)
-		(stroke
-			(width 0)
-			(type default)
-		)
-	)
-	(wire
-		(pts
-			(xy 57.15 67.31) (xy 80.01 67.31)
+			(xy 80.01 45.72) (xy 80.01 64.77)
+		)
+		(stroke
+			(width 0)
+			(type default)
+		)
+	)
+	(wire
+		(pts
+			(xy 62.23 59.69) (xy 58.42 59.69)
+		)
+		(stroke
+			(width 0)
+			(type default)
+		)
+	)
+	(wire
+		(pts
+			(xy 97.79 40.64) (xy 128.27 40.64)
+		)
+		(stroke
+			(width 0)
+			(type default)
+		)
+	)
+	(wire
+		(pts
+			(xy 58.42 59.69) (xy 58.42 64.77)
+		)
+		(stroke
+			(width 0)
+			(type default)
+		)
+	)
+	(wire
+		(pts
+			(xy 35.56 67.31) (xy 43.18 67.31)
 		)
 		(stroke
@@
 	(wire
 		(pts
+			(xy 80.01 64.77) (xy 58.42 64.77)
+		)
+		(stroke
+			(width 0)
+			(type default)
+		)
+	)
+	(wire
+		(pts
 			(xy 111.76 78.74) (xy 102.87 78.74)
 		)
@@
 	(wire
 		(pts
-			(xy 57.15 35.56) (xy 57.15 39.37)
-		)
-		(stroke
-			(width 0)
-			(type default)
-		)
-	)
-	(wire
-		(pts
-			(xy 57.15 35.56) (xy 80.01 35.56)
+			(xy 62.23 35.56) (xy 62.23 38.1)
+		)
+		(stroke
+			(width 0)
+			(type default)
+		)
+	)
+	(wire
+		(pts
+			(xy 128.27 40.64) (xy 128.27 62.23)
+		)
+		(stroke
+			(width 0)
+			(type default)
+		)
+	)
+	(wire
+		(pts
+			(xy 62.23 35.56) (xy 80.01 35.56)
 		)
 		(stroke
@@
 	)
 	(label "Shutter_Output"
-		(at 36.83 67.31 0)
+		(at 36.83 55.88 0)
 		(fields_autoplaced yes)
 		(effects
@@
 		(on_board yes)
 		(dnp no)
-		(fields_autoplaced yes)
 		(property "Reference" "R1"
 			(at 119.38 55.88 90)
@@
 	(symbol
 		(lib_id "Device:R_US")
-		(at 57.15 57.15 0)
+		(at 62.23 55.88 0)
 		(unit 1)
 		(exclude_from_sim no)
@@
 		(dnp no)
 		(property "Reference" "R6"
-			(at 59.69 55.8799 0)
+			(at 64.77 54.6099 0)
 			(effects
 				(font
@@
 		)
 		(property "Value" "36K"
-			(at 59.69 58.4199 0)
+			(at 64.77 57.1499 0)
 			(effects
 				(font
@@
 		)
 		(property "Footprint" "Resistor_THT:R_Axial_DIN0204_L3.6mm_D1.6mm_P7.62mm_Horizontal"
-			(at 58.166 57.404 90)
+			(at 63.246 56.134 90)
 			(effects
 				(font
@@
 		)
 		(property "Datasheet" "~"
-			(at 57.15 57.15 0)
+			(at 62.23 55.88 0)
 			(effects
 				(font
@@
 		)
 		(property "Description" "Resistor, US symbol"
-			(at 57.15 57.15 0)
+			(at 62.23 55.88 0)
 			(effects
 				(font
@@
 	(symbol
 		(lib_id "Device:R_US")
-		(at 57.15 43.18 0)
+		(at 62.23 41.91 0)
 		(unit 1)
 		(exclude_from_sim no)
@@
 		(dnp no)
 		(property "Reference" "R5"
-			(at 59.69 41.9099 0)
+			(at 64.77 40.6399 0)
 			(effects
 				(font
@@
 		)
 		(property "Value" "2,9K"
-			(at 59.69 44.4499 0)
+			(at 64.77 43.1799 0)
 			(effects
 				(font
@@
 		)
 		(property "Footprint" "Resistor_THT:R_Axial_DIN0204_L3.6mm_D1.6mm_P7.62mm_Horizontal"
-			(at 58.166 43.434 90)
+			(at 63.246 42.164 90)
 			(effects
 				(font
@@
 		)
 		(property "Datasheet" "~"
-			(at 57.15 43.18 0)
+			(at 62.23 41.91 0)
 			(effects
 				(font
@@
 		)
 		(property "Description" "Resistor, US symbol"
-			(at 57.15 43.18 0)
+			(at 62.23 41.91 0)
 			(effects
 				(font
@@
 	)
 	(symbol
-		(lib_id "Connector:TestPoint")
-		(at 156.21 40.64 270)
-		(unit 1)
-		(exclude_from_sim no)
-		(in_bom yes)
-		(on_board yes)
-		(dnp no)
-		(fields_autoplaced yes)
-		(property "Reference" "TP7"
-			(at 161.29 39.3699 90)
-			(effects
-				(font
-					(size 1.27 1.27)
-				)
-				(justify left)
-			)
-		)
-		(property "Value" "S2"
-			(at 161.29 41.9099 90)
-			(effects
-				(font
-					(size 1.27 1.27)
-				)
-				(justify left)
-			)
-		)
-		(property "Footprint" "TestPoint:TestPoint_THTPad_2.0x2.0mm_Drill1.0mm"
-			(at 156.21 45.72 0)
+		(lib_id "Switch:SW_DIP_x02")
+		(at 50.8 67.31 0)
+		(mirror y)
+		(unit 1)
+		(exclude_from_sim no)
+		(in_bom yes)
+		(on_board yes)
+		(dnp no)
+		(property "Reference" "SW1"
+			(at 50.8 74.93 0)
+			(effects
+				(font
+					(size 1.27 1.27)
+				)
+			)
+		)
+		(property "Value" "SW_DIP_x02"
+			(at 50.8 72.39 0)
+			(effects
+				(font
+					(size 1.27 1.27)
+				)
+			)
+		)
+		(property "Footprint" "Button_Switch_THT:SW_DIP_SPSTx02_Slide_9.78x7.26mm_W7.62mm_P2.54mm"
+			(at 50.8 67.31 0)
 			(effects
 				(font
@@
 		)
 		(property "Datasheet" "~"
-			(at 156.21 45.72 0)
-			(effects
-				(font
-					(size 1.27 1.27)
-				)
-				(hide yes)
-			)
-		)
-		(property "Description" "test point"
-			(at 156.21 40.64 0)
-			(effects
-				(font
-					(size 1.27 1.27)
-				)
-				(hide yes)
-			)
-		)
-		(pin "1"
-		)
-		(instances
-			(project "canon+GH4"
-				(path "/923b77b9-2deb-4a0b-afd3-30df7d2956a6"
-					(reference "TP7")
-					(unit 1)
-				)
+			(at 50.8 67.31 0)
+			(effects
+				(font
+					(size 1.27 1.27)
+				)
+				(hide yes)
+			)
+		)
+		(property "Description" "2x DIP Switch, Single Pole Single Throw (SPST) switch, small symbol"
+			(at 50.8 67.31 0)
+			(effects
+				(font
+					(size 1.27 1.27)
+				)
+				(hide yes)
+			)
+		)
+		(pin "2"
+		)
+		(pin "4"
+		)
+		(pin "1"
+		)
+		(pin "3"
+		)
+		(instances
+			(project ""
+				(path "/923b77b9-2deb-4a0b-afd3-30df7d2956a6"
+					(reference "SW1")
+					(unit 1)
+				)
